File: KiCAD model/Lab1.sch (KiCad schematic (older format))
At the start: 116 parts, among them J1 USB_OTG, J2 SWD, SW1 1825910-6, SW10 Rotary_Encoder, U1 PMW3389, U2 AP2125N-3.3TRG, U3 MIC5235YM5-TR, U4 STM32F411RETx, U5 USBLC6-2SC6, Y1 16Mhz

Commit message: final pcb design
Parts:
- removed D1, D2, D3, D4, D5, D6: Indicator LED, LED_SMD:LED_1206_3216Metric, symbol LED:IR26-21C_L110_TR8
- removed JP2, JP3, JP4: DFU, Connector:FanPinHeader_1x03_P2.54mm_Vertical, symbol Jumper:Jumper_3_Bridged12
- removed R1: 47, Resistor_SMD:R_0805_2012Metric_Pad1.20x1.40mm_HandSolder, symbol Device:R
- removed R14, R17, R18, R22: 10k, Resistor_SMD:R_0805_2012Metric_Pad1.20x1.40mm_HandSolder, symbol Device:R
- removed R15, R16, R21: 150, Resistor_SMD:R_0805_2012Metric_Pad1.20x1.40mm_HandSolder, symbol Device:R
- removed R5: 820, Resistor_SMD:R_0805_2012Metric_Pad1.20x1.40mm_HandSolder, symbol Device:R
- removed R6: 1.5k, Resistor_SMD:R_0805_2012Metric_Pad1.20x1.40mm_HandSolder, symbol Device:R
- removed S2, S3, S4, S5, S6, S7: D2F-FL, Desktop:SW_D2F-FL, symbol D2F-FL:D2F-FL
- removed TP16: wheel_click, TestPoint:TestPoint_Pad_1.5x1.5mm, symbol Connector:TestPoint
- added D4: LED_ABGR, Components:LED_RGB_1210_RND_135-00251, symbol Device:LED_ABGR
- added S2, S3, S4, S5, S6, S7: D2F-FL, Components:SW_D2F-FL, symbol Lab1-rescue:D2F-FL-D2F-FL
- added TP15: TestPoint, TestPoint:TestPoint_Pad_1.5x1.5mm, symbol Connector:TestPoint
- C10, C11, C12, C13, C14, C9: value 1u -> 100n
- J1: footprint Connector_USB:USB_Mini-B_Tensility_54-00023_Vertical -> Connector_USB:USB_Micro-B_Wuerth_614105150721_Vertical
- J2: footprint Connector_PinHeader_2.00mm:PinHeader_1x06_P2.00mm_Vertical -> Connector_PinHeader_2.54mm:PinHeader_1x06_P2.54mm_Vertical
- JP1: footprint Connector:FanPinHeader_1x03_P2.54mm_Vertical -> Connector_PinHeader_2.54mm:PinHeader_1x03_P2.54mm_Vertical
- R10, R13, R9: value 10k -> 1k
- R11, R12, R7, R8: value 150 -> 1k
- S1: footprint Desktop:SW_D2F-FL -> Components:SW_D2F-FL; symbol D2F-FL:D2F-FL -> Lab1-rescue:D2F-FL-D2F-FL
- SW1: footprint Desktop:SW_1825910-6-4 -> Components:SW_1825910-6-4; symbol 1825910-6:1825910-6 -> Lab1-rescue:1825910-6-1825910-6
- SW10: footprint Custom:PEC12R-2120F-N0012 -> Components:EC10E1220505
- U2: footprint Package_TO_SOT_SMD:TO-252-3_TabPin2 -> Package_TO_SOT_SMD:SOT-23_Handsoldering
- U3: footprint Package_TO_SOT_SMD:SOT-23-5 -> Package_TO_SOT_SMD:SOT-23-5_HandSoldering
- Y1: footprint Crystal:Crystal_SMD_0603-2Pin_6.0x3.5mm_HandSoldering -> Crystal:Crystal_SMD_HC49-SD_HandSoldering
Connections:
- net +3V3: now also S1.NO, D4.1 (A), S2.NO, S3.NO, S4.NO, S5.NO, S6.NO, S7.NO; no longer R10.1, R13.1, R9.1
- net GND: now also S1.NC, S2.NC, S3.NC, S4.NC, S5.NC, S6.NC, S7.NC; no longer S1.NO
- net backward: now also C26.1, R11.2, TP12.1; no longer C27.1, TP13.1
- net forward: now also C25.1, R10.2, TP11.1; no longer C26.1, TP12.1
- net left_click: now also C23.1, TP9.1; no longer C22.1, TP5.1
- net right_click: now also C22.1, R9.2, TP5.1; no longer C23.1, R8.2, TP9.1
- net sense_down: now also C27.1, TP13.1; no longer C25.1, TP11.1
- net sense_up: now also R8.2; no longer R11.2
- net wheel_click: now also R13.2, TP15.1
- net at R8.1: now also S3.COM; no longer R10.2
- net at R11.1: now also S5.COM; no longer R13.2
- net at R12.1: now also S6.COM
- net at R24.1: now also D4.4 (RK)
- net at R25.1: now also D4.3 (GK)
- net at R26.1: now also D4.2 (BK)
- new net: R9.1, S1.COM
- new net: R10.1, S4.COM
- new net: R13.1, S7.COM
- new net: R7.1, S2.COM
- no-connect marks 38 -> 31
Other:
- note removed: "BLUE"
- note removed: "GREEN"
- note removed: "RED"
- moved on the sheet: C22, R24, R25, R26, R9, S1, TP5
