File: KiCAD model/Lab1.kicad_pcb (KiCad board)
At the start: 2 copper layers, 50 x 80 mm, 116 parts, among them J1 USB_OTG, J2 SWD, SW1 1825910-6, SW10 Rotary_Encoder, U1 PMW3389, U2 AP2125N-3.3TRG, U3 MIC5235YM5-TR, U4 STM32F411RETx, U5 USBLC6-2SC6, Y1 16Mhz

Commit message: final pcb design
Parts:
- removed D1, D2, D3, D5, D6: Indicator LED, LED_SMD:LED_1206_3216Metric
- removed JP2, JP3, JP4: DFU, Connector:FanPinHeader_1x03_P2.54mm_Vertical
- removed R1: 47, Resistor_SMD:R_0805_2012Metric_Pad1.20x1.40mm_HandSolder
- removed R14, R17, R18, R22: 10k, Resistor_SMD:R_0805_2012Metric_Pad1.20x1.40mm_HandSolder
- removed R15, R16, R21: 150, Resistor_SMD:R_0805_2012Metric_Pad1.20x1.40mm_HandSolder
- removed R5: 820, Resistor_SMD:R_0805_2012Metric_Pad1.20x1.40mm_HandSolder
- removed R6: 1.5k, Resistor_SMD:R_0805_2012Metric_Pad1.20x1.40mm_HandSolder
- removed TP16: wheel_click, TestPoint:TestPoint_Pad_1.5x1.5mm
- added TP15: TestPoint, TestPoint:TestPoint_Pad_1.5x1.5mm, F.Cu at (70.6, 51.2)
- C10, C11, C12, C13, C14, C9: value 1u -> 100n
- D4: value Indicator LED -> LED_ABGR; footprint LED_SMD:LED_1206_3216Metric -> Components:LED_RGB_1210_RND_135-00251
- J1: footprint Connector_USB:USB_Mini-B_Tensility_54-00023_Vertical -> Connector_USB:USB_Micro-B_Wuerth_614105150721_Vertical
- J2: footprint Connector_PinHeader_2.00mm:PinHeader_1x06_P2.00mm_Vertical -> Connector_PinHeader_2.54mm:PinHeader_1x06_P2.54mm_Vertical
- JP1: footprint Connector:FanPinHeader_1x03_P2.54mm_Vertical -> Connector_PinHeader_2.54mm:PinHeader_1x03_P2.54mm_Vertical
- R10, R13, R9: value 10k -> 1k
- R11, R12, R7, R8: value 150 -> 1k
- S1, S2, S3, S4, S5, S6, S7: footprint Desktop:SW_D2F-FL -> Components:SW_D2F-FL
- SW1: footprint Desktop:SW_1825910-6-4 -> Components:SW_1825910-6-4
- SW10: footprint Custom:PEC12R-2120F-N0012 -> Components:EC10E1220505
- U2: footprint Package_TO_SOT_SMD:TO-252-3_TabPin2 -> Package_TO_SOT_SMD:SOT-23_Handsoldering
- U3: footprint Package_TO_SOT_SMD:SOT-23-5 -> Package_TO_SOT_SMD:SOT-23-5_HandSoldering
- Y1: footprint Crystal:Crystal_SMD_0603-2Pin_6.0x3.5mm_HandSoldering -> Crystal:Crystal_SMD_HC49-SD_HandSoldering
- moved TP6 170.6 mm to (34.5, 54.4)
- moved C3 167.8 mm to (37.9, 44.0)
- moved TP9 166.7 mm to (38.8, 40.6)
- moved TP27 163.6 mm to (51.0, 105.5)
- moved C4 163.4 mm to (37.9, 56.1)
- moved C2 162.1 mm to (33.9, 52.0), turned to 180 degrees
- moved TP26 161.9 mm to (48.5, 106.6)
- moved TP11 158.4 mm to (43.6, 83.4)
- moved C18 158.2 mm to (44.5, 64.9), turned to 270 degrees
- moved C11 156.0 mm to (43.2, 104.1), turned to 90 degrees
- moved C26 153.0 mm to (40.6, 75.9), turned to 90 degrees
- moved C20 152.2 mm to (45.6, 72.1)
- moved TP19 150.7 mm to (34.5, 57.0)
- moved TP1 148.3 mm to (31.6, 32.0)
- moved C25 145.8 mm to (40.6, 67.9), turned to 90 degrees
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Connections:
- C22 pad 1: left_click -> right_click
- C23 pad 1: right_click -> left_click
- C25 pad 1: sense_down -> forward
- C26 pad 1: forward -> backward
- C27 pad 1: backward -> sense_down
- D4 pad 1: GND -> +3V3
- R10 pad 1: +3V3 -> Net-(R10-Pad1)
- R10 pad 2: Net-(R10-Pad2) -> forward
- R11 pad 2: sense_up -> backward
- R13 pad 1: +3V3 -> Net-(R13-Pad1)
- R13 pad 2: Net-(R11-Pad1) -> wheel_click
- R24 pad 1: Net-(D4-Pad2) -> Net-(D4-Pad4)
- R25 pad 1: Net-(D5-Pad2) -> Net-(D4-Pad3)
- R26 pad 1: Net-(D6-Pad2) -> Net-(D4-Pad2)
- R8 pad 1: Net-(R10-Pad2) -> Net-(R8-Pad1)
- R8 pad 2: right_click -> sense_up
- R9 pad 1: +3V3 -> Net-(R9-Pad1)
- R9 pad 2: Net-(R7-Pad1) -> right_click
- S1 pad COM: Net-(R7-Pad1) -> Net-(R9-Pad1)
- S1 pad NC: Net-(S1-PadNC) -> GND
- S1 pad NO: GND -> +3V3
- S2 pad COM: Net-(R10-Pad2) -> Net-(R7-Pad1)
- S2 pad NC: Net-(S2-PadNC) -> GND
- S2 pad NO: GND -> +3V3
- S3 pad COM: Net-(R11-Pad1) -> Net-(R8-Pad1)
- S3 pad NC: Net-(S3-PadNC) -> GND
- S3 pad NO: GND -> +3V3
- S4 pad COM: Net-(R12-Pad1) -> Net-(R10-Pad1)
- S4 pad NC: Net-(S4-PadNC) -> GND
- S4 pad NO: GND -> +3V3
- S5 pad COM: Net-(R15-Pad1) -> Net-(R11-Pad1)
- S5 pad NC: Net-(S5-PadNC) -> GND
- S5 pad NO: GND -> +3V3
- S6 pad COM: Net-(R16-Pad1) -> Net-(R12-Pad1)
- S6 pad NC: Net-(S6-PadNC) -> GND
- S6 pad NO: GND -> +3V3
- S7 pad COM: Net-(R21-Pad1) -> Net-(R13-Pad1)
- S7 pad NC: Net-(S7-PadNC) -> GND
- S7 pad NO: GND -> +3V3
- TP11 pad 1: sense_down -> forward
- TP12 pad 1: forward -> backward
- TP13 pad 1: backward -> sense_down
- TP5 pad 1: left_click -> right_click
- TP9 pad 1: right_click -> left_click
Routing:
- net GND: track 0.00 -> 355.7 mm, vias 0 -> 22
- net +3V3: track 0.00 -> 293.1 mm, vias 0 -> 22
- net +5V: track 0.00 -> 141.2 mm, vias 0 -> 4
- net right_click: track 0.00 -> 124.8 mm, vias 0 -> 6
- net Scroll_b: track 0.00 -> 121.5 mm, vias 0 -> 2
- net RED: track 0.00 -> 116.0 mm, vias 0 -> 2
- net wheel_click: track 0.00 -> 113.8 mm, vias 0 -> 2
- net sense_down: track 0.00 -> 112.5 mm, vias 0 -> 2
- net Scroll_a: track 0.00 -> 106.8 mm, vias 0 -> 2
- net Motion: track 0.00 -> 99.3 mm, vias 0 -> 2
- net NRST: track 0.00 -> 94.0 mm, vias 0 -> 4
- net left_click: track 0.00 -> 92.1 mm, vias 0 -> 4
- net SCK: track 0.00 -> 89.6 mm
- net sense_up: track 0.00 -> 88.6 mm
- net BLUE: track 0.00 -> 87.0 mm
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- added copper zone on B.Cu, net GND
- added copper zone on F.Cu, net GND
Other:
- outline, holes or cut-outs redrawn

Commit message: fix swdio/swclk + usb issue
Parts:
- turned S2 to 180 degrees
Connections:
- U4 pad 43: OUT_D- -> Scroll_a
- U4 pad 44: OUT_D+ -> OUT_D-
- U4 pad 45: SWDIO -> OUT_D+
- U4 pad 46: SWCLK -> SWDIO
- U4 pad 49: Scroll_a -> SWCLK
Routing:
- net GND: track 355.7 -> 335.5 mm
- net Net-(R7-Pad1): track 5.75 -> 13.9 mm
- net Scroll_a: track 106.8 -> 114.3 mm, vias 2 -> 4
- net SWCLK: track 23.5 -> 29.0 mm, vias 0 -> 4
- net SWDIO: track 28.2 -> 27.5 mm
- net +3V3: track 293.1 -> 293.7 mm
